File: hardware/HDW_HACKABLE_LAMP.kicad_sch (KiCad schematic)
At the start: 0 parts

Commit message: added ESP32 and WS2812
Parts:
- added D1, D10, D11, D12, D13, D14, D15, D16, D17, D18, D19, D2, D20, D21, D22, D23, D24, D3, D4, D5, D6, D7, D8, D9: WS2812B, LED_SMD:LED_WS2812B_PLCC4_5.0x5.0mm_P3.2mm, symbol LED:WS2812B
- added U1: ESP32-WROOM-32E, RF_Module:ESP32-WROOM-32D, symbol RF_Module:ESP32-WROOM-32E
Connections:
- new net: D10.2 (DOUT), D11.4 (DIN)
- new net: D10.4 (DIN), D9.2 (DOUT)
- new net: D19.2 (DOUT), D20.4 (DIN)
- new net: D18.2 (DOUT), D19.4 (DIN)
- new net: D2.2 (DOUT), D3.4 (DIN)
- new net: D1.2 (DOUT), D2.4 (DIN)
- new net: D23.2 (DOUT), D24.4 (DIN)
- new net: D22.2 (DOUT), D23.4 (DIN)
- new net: D17.2 (DOUT), D18.4 (DIN)
- new net: D11.2 (DOUT), D12.4 (DIN)
- new net: D3.2 (DOUT), D4.4 (DIN)
- new net: D21.2 (DOUT), D22.4 (DIN)
- new net: D20.2 (DOUT), D21.4 (DIN)
- new net: D6.2 (DOUT), D7.4 (DIN)
- new net: D5.2 (DOUT), D6.4 (DIN)
- new net: D13.2 (DOUT), D14.4 (DIN)
- new net: D8.2 (DOUT), D9.4 (DIN)
- new net: D4.2 (DOUT), D5.4 (DIN)
- new net: D16.2 (DOUT), D17.4 (DIN)
- new net: D7.2 (DOUT), D8.4 (DIN)
- new net: D14.2 (DOUT), D15.4 (DIN)
- new net: D15.2 (DOUT), D16.4 (DIN)
- new net: U1.1 (GND), U1.15 (GND), U1.38 (GND), U1.39 (GND)
- new net GND: D1.3 (VSS), D10.3 (VSS), D11.3 (VSS), D12.3 (VSS), D13.3 (VSS), D14.3 (VSS), D15.3 (VSS), D16.3 (VSS), D17.3 (VSS), D18.3 (VSS), D19.3 (VSS), D2.3 (VSS), D20.3 (VSS), D21.3 (VSS), D22.3 (VSS), D23.3 (VSS), D24.3 (VSS), D3.3 (VSS), D4.3 (VSS), D5.3 (VSS), D6.3 (VSS), D7.3 (VSS), D8.3 (VSS), D9.3 (VSS)
- new net VDD: D1.1 (VDD), D10.1 (VDD), D11.1 (VDD), D12.1 (VDD), D13.1 (VDD), D14.1 (VDD), D15.1 (VDD), D16.1 (VDD), D17.1 (VDD), D18.1 (VDD), D19.1 (VDD), D2.1 (VDD), D20.1 (VDD), D21.1 (VDD), D22.1 (VDD), D23.1 (VDD), D24.1 (VDD), D3.1 (VDD), D4.1 (VDD), D5.1 (VDD), D6.1 (VDD), D7.1 (VDD), D8.1 (VDD), D9.1 (VDD)
